File: PCB/hackboard.kicad_pcb (KiCad board)
At the start: 2 copper layers, 474.9 x 141 mm, 205 parts, among them SW1 SW_Push_45deg, SW10 SW_Push_45deg, SW100 SW_Push_45deg, SW101 SW_Push_45deg, SW102 SW_Push_45deg, SW103 SW_Push_45deg, SW104 SW_Push_45deg, SW11 SW_Push_45deg, SW12 SW_Push_45deg, SW13 SW_Push_45deg, SW17 SW_Push_45deg, SW18 SW_Push_45deg, SW19 SW_Push_45deg, SW2 SW_Push_45deg, SW20 SW_Push_45deg, SW21 SW_Push_45deg, SW22 SW_Push_45deg, SW23 SW_Push_45deg, SW24 SW_Push_45deg, SW25 SW_Push_45deg, SW26 SW_Push_45deg, SW27 SW_Push_45deg, SW28 SW_Push_45deg, SW29 SW_Push_45deg, SW3 SW_Push_45deg, SW30 SW_Push_45deg, SW31 SW_Push_45deg, SW32 SW_Push_45deg, SW33 SW_Push_45deg, SW34 SW_Push_45deg, SW35 SW_Push_45deg, SW36 SW_Push_45deg, SW37 SW_Push_45deg, SW38 SW_Push_45deg, SW39 SW_Push_45deg, SW4 SW_Push_45deg, SW40 SW_Push_45deg, SW41 SW_Push_45deg, SW42 SW_Push_45deg, SW43 SW_Push_45deg, SW44 SW_Push_45deg, SW45 SW_Push_45deg, SW46 SW_Push_45deg, SW47 SW_Push_45deg, SW48 SW_Push_45deg, SW49 SW_Push_45deg, SW5 SW_Push_45deg, SW50 SW_Push_45deg, SW51 SW_Push_45deg, SW52 SW_Push_45deg, SW53 SW_Push_45deg, SW54 SW_Push_45deg, SW55 SW_Push_45deg, SW56 SW_Push_45deg, SW57 SW_Push_45deg, SW58 SW_Push_45deg, SW59 SW_Push_45deg, SW6 SW_Push_45deg, SW60 SW_Push_45deg, SW61 SW_Push_45deg, SW62 SW_Push_45deg, SW63 SW_Push_45deg, SW64 SW_Push_45deg, SW65 SW_Push_45deg, SW66 SW_Push_45deg, SW67 SW_Push_45deg, SW68 SW_Push_45deg, SW69 SW_Push_45deg, SW7 SW_Push_45deg, SW70 SW_Push_45deg, SW71 SW_Push_45deg, SW72 SW_Push_45deg, SW73 SW_Push_45deg, SW74 SW_Push_45deg, SW75 SW_Push_45deg, SW76 SW_Push_45deg, SW77 SW_Push_45deg, SW78 SW_Push_45deg, SW79 SW_Push_45deg, SW8 SW_Push_45deg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

Commit message: Add files via upload
Parts:
- removed D100, D101, D102, D103, D104, D96, D97, D98, D99: 1N4148, Diode_SMD:D_SOD-123
- removed SW100, SW101, SW102, SW104: SW_Push_45deg, Button_Switch_Keyboard:SW_Cherry_MX_1.00u_PCB
- removed SW103: SW_Push_45deg, Button_Switch_Keyboard:SW_Cherry_MX_2.00u_PCB
- removed SW96: SW_Push_45deg, Button_Switch_Keyboard:SW_Cherry_MX_6.25u_PCB
- removed SW97, SW98, SW99: SW_Push_45deg, Button_Switch_Keyboard:SW_Cherry_MX_1.25u_PCB
- added D14: 1N4148, Diode_SMD:D_SOD-123, B.Cu at (352.8, 91.2)
- added D15: 1N4148, Diode_SMD:D_SOD-123, B.Cu at (371.9, 91.2)
- added D16: 1N4148, Diode_SMD:D_SOD-123, B.Cu at (390.9, 91.2)
- added SW14: SW_Push_45deg, Button_Switch_Keyboard:SW_Cherry_MX_1.00u_PCB, F.Cu at (364.6, 84.6)
- added SW15: SW_Push_45deg, Button_Switch_Keyboard:SW_Cherry_MX_1.00u_PCB, F.Cu at (383.6, 84.6)
- added SW16: SW_Push_45deg, Button_Switch_Keyboard:SW_Cherry_MX_1.00u_PCB, F.Cu at (402.7, 84.6)
- SW1: value SW_Push_45deg -> RotaryEncoder_Switch; footprint Button_Switch_Keyboard:SW_Cherry_MX_1.00u_PCB -> Rotary_Encoder:RotaryEncoder_Alps_EC11E-Switch_Vertical_H20mm
- SW30: footprint Button_Switch_Keyboard:SW_Cherry_MX_2.00u_PCB -> Button_Switch_Keyboard:SW_Cherry_MX_1.00u_PCB
- SW32, SW81: footprint Button_Switch_Keyboard:SW_Cherry_MX_1.00u_PCB -> Button_Switch_Keyboard:SW_Cherry_MX_2.00u_PCB
- SW35, SW48: footprint Button_Switch_Keyboard:SW_Cherry_MX_1.00u_PCB -> Button_Switch_Keyboard:SW_Cherry_MX_1.50u_PCB
- SW38: footprint Button_Switch_Keyboard:SW_Cherry_MX_1.50u_PCB -> Button_Switch_Keyboard:SW_Cherry_MX_1.00u_PCB
- SW51: footprint Button_Switch_Keyboard:SW_Cherry_MX_1.50u_PCB -> Button_Switch_Keyboard:SW_Cherry_MX_2.00u_Vertical_PCB
- SW52, SW79: footprint Button_Switch_Keyboard:SW_Cherry_MX_1.00u_PCB -> Button_Switch_Keyboard:SW_Cherry_MX_1.75u_PCB
- SW58: footprint Button_Switch_Keyboard:SW_Cherry_MX_2.00u_Vertical_PCB -> Button_Switch_Keyboard:SW_Cherry_MX_1.00u_PCB
- SW59: footprint Button_Switch_Keyboard:SW_Cherry_MX_1.75u_PCB -> Button_Switch_Keyboard:SW_Cherry_MX_1.00u_PCB
- SW64, SW68: footprint Button_Switch_Keyboard:SW_Cherry_MX_1.00u_PCB -> Button_Switch_Keyboard:SW_Cherry_MX_2.25u_PCB
- SW71, SW75: footprint Button_Switch_Keyboard:SW_Cherry_MX_2.25u_PCB -> Button_Switch_Keyboard:SW_Cherry_MX_1.00u_PCB
- SW84: footprint Button_Switch_Keyboard:SW_Cherry_MX_1.00u_PCB -> Button_Switch_Keyboard:SW_Cherry_MX_2.00u_Vertical_PCB
- SW85, SW90: footprint Button_Switch_Keyboard:SW_Cherry_MX_1.00u_PCB -> Button_Switch_Keyboard:SW_Cherry_MX_1.25u_PCB
- SW86: footprint Button_Switch_Keyboard:SW_Cherry_MX_2.75u_PCB -> Button_Switch_Keyboard:SW_Cherry_MX_1.00u_PCB
- SW89: footprint Button_Switch_Keyboard:SW_Cherry_MX_1.00u_PCB -> Button_Switch_Keyboard:SW_Cherry_MX_6.25u_PCB
- SW91: footprint Button_Switch_Keyboard:SW_Cherry_MX_2.00u_Vertical_PCB -> Button_Switch_Keyboard:SW_Cherry_MX_1.25u_PCB
- SW92, SW93, SW94, SW95: footprint Button_Switch_Keyboard:SW_Cherry_MX_1.25u_PCB -> Button_Switch_Keyboard:SW_Cherry_MX_1.00u_PCB
- moved D34 377.4 mm to (95.6, 129.3)
- moved SW34 377.4 mm to (107.4, 122.7)
- moved D33 372.6 mm to (76.6, 129.3)
- moved SW33 372.6 mm to (88.3, 122.7)
- moved D1 351.6 mm to (467.1, 95.6)
- moved D35 330.0 mm to (162.3, 129.3)
- moved SW35 325.2 mm to (178.8, 122.7)
- moved SW1 322.5 mm to (449.9, 86.7)
- moved D37 320.5 mm to (209.9, 129.3)
- moved SW36 320.5 mm to (202.6, 122.7)
- moved D36 320.5 mm to (190.9, 129.3)
- moved SW37 320.5 mm to (221.7, 122.7)
- moved D92 295.7 mm to (410.0, 186.5)
- moved SW92 293.4 mm to (421.7, 179.9)
- moved D93 291.1 mm to (429.0, 186.5)
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Connections:
- D31 pad 1: row 1 -> row 2
- D32 pad 1: row 1 -> row 2
- D33 pad 1: row 1 -> row 3
- D37 pad 1: row 1 -> row 3
- D49 pad 1: row 3 -> row 4
- D50 pad 1: row 3 -> row 4
- D51 pad 1: row 3 -> row 4
- D52 pad 1: row 2 -> row 4
- D53 pad 1: row 2 -> row 4
- D54 pad 1: row 2 -> row 4
- D58 pad 1: row 2 -> row 4
- D65 pad 1: row 4 -> row 5
- D66 pad 1: row 4 -> row 5
- D67 pad 1: row 4 -> row 5
- D68 pad 1: row 4 -> row 5
- D69 pad 1: row 4 -> row 5
- D70 pad 1: row 4 -> row 5
- D71 pad 1: row 4 -> row 5
- D74 pad 1: row 3 -> row 5
- D81 pad 1: row 5 -> row 6
- D82 pad 1: row 5 -> row 6
- D83 pad 1: row 5 -> row 6
- D84 pad 1: row 5 -> row 6
- D85 pad 1: row 5 -> row 6
- D86 pad 1: row 5 -> row 6
- D87 pad 1: row 4 -> row 6
- D91 pad 1: row 4 -> row 6
- SW10 pad 1: col 10 -> col 9
- SW11 pad 1: col 11 -> col 10
- SW12 pad 1: col 12 -> col 11
- SW13 pad 1: col 13 -> col 12
- SW2 pad 1: col 2 -> col 1
- SW3 pad 1: col 3 -> col 2
- SW33 pad 1: col 17 -> col 1
- SW34 pad 1: col 15 -> col 2
- SW35 pad 1: col 16 -> col 3
- SW36 pad 1: col 17 -> col 4
- SW37 pad 1: col 18 -> col 5
- SW38 pad 1: col 1 -> col 6
- SW39 pad 1: col 2 -> col 7
- SW4 pad 1: col 4 -> col 3
- SW40 pad 1: col 3 -> col 8
- SW41 pad 1: col 4 -> col 9
- SW42 pad 1: col 5 -> col 10
- SW43 pad 1: col 6 -> col 11
- SW44 pad 1: col 7 -> col 12
- SW45 pad 1: col 8 -> col 13
- SW46 pad 1: col 9 -> col 14
- SW47 pad 1: col 10 -> col 15
- SW48 pad 1: col 11 -> col 16
- SW49 pad 1: col 12 -> col 1
- SW5 pad 1: col 5 -> col 4
- SW50 pad 1: col 13 -> col 2
- SW51 pad 1: col 14 -> col 3
- SW52 pad 1: col 15 -> col 4
- SW53 pad 1: col 16 -> col 5
- SW54 pad 1: col 17 -> col 6
- SW55 pad 1: col 15 -> col 7
- SW56 pad 1: col 16 -> col 8
- SW57 pad 1: col 17 -> col 9
- SW58 pad 1: col 18 -> col 10
- SW59 pad 1: col 1 -> col 11
- SW6 pad 1: col 6 -> col 5
- SW60 pad 1: col 2 -> col 12
- SW61 pad 1: col 3 -> col 13
- SW62 pad 1: col 4 -> col 14
- SW63 pad 1: col 5 -> col 15
- SW64 pad 1: col 6 -> col 16
- SW65 pad 1: col 7 -> col 1
- SW66 pad 1: col 8 -> col 2
- SW67 pad 1: col 9 -> col 3
- SW68 pad 1: col 10 -> col 4
- SW69 pad 1: col 11 -> col 5
- SW7 pad 1: col 7 -> col 6
- SW70 pad 1: col 12 -> col 6
- SW71 pad 1: col 13 -> col 7
- SW72 pad 1: col 15 -> col 8
- SW73 pad 1: col 16 -> col 9
- SW74 pad 1: col 18 -> col 10
- SW75 pad 1: col 1 -> col 11
- SW76 pad 1: col 3 -> col 12
- SW77 pad 1: col 4 -> col 13
- SW78 pad 1: col 5 -> col 14
- SW79 pad 1: col 6 -> col 15
- SW8 pad 1: col 8 -> col 7
- SW80 pad 1: col 7 -> col 16
- SW81 pad 1: col 8 -> col 1
- SW82 pad 1: col 9 -> col 2
- SW83 pad 1: col 10 -> col 3
- SW84 pad 1: col 11 -> col 4
- SW85 pad 1: col 12 -> col 5
- SW86 pad 1: col 13 -> col 6
- SW87 pad 1: col 14 -> col 7
- SW88 pad 1: col 15 -> col 8
- SW89 pad 1: col 16 -> col 10
- SW9 pad 1: col 9 -> col 8
- SW90 pad 1: col 17 -> col 11
- SW91 pad 1: col 18 -> col 12
- SW92 pad 1: col 1 -> col 13
- SW93 pad 1: col 3 -> col 14
- SW94 pad 1: col 4 -> col 15
- SW95 pad 1: col 5 -> col 16
- U1 pad 1: data -> row 6
- U1 pad 10: col 11 -> col 2
- U1 pad 12: col 9 -> col 11
- U1 pad 14: col 16 -> col 4
- U1 pad 15: col 8 -> col 5
- U1 pad 16: row 3 -> col 6
- U1 pad 17: row 4 -> col 7
- U1 pad 19: row 5 -> col 8
- U1 pad 2: clock -> col 1
- U1 pad 20: row 6 -> col 9
- U1 pad 21: col 17 -> col 16
- U1 pad 22: col 2 -> col 15
- U1 pad 24: row 2 -> col 14
- U1 pad 25: col 5 -> col 13
- U1 pad 26: col 6 -> col 12
- U1 pad 27: col 7 -> col 3
- U1 pad 28: unconnected-(U1-GND-Pad28) -> GND
- U1 pad 29: col 4 -> encA
- U1 pad 31: col 3 -> data
- U1 pad 32: row 1 -> clock
- U1 pad 34: col 1 -> encB
- U1 pad 38: GND -> unconnected-(U1-GND-Pad38)
- U1 pad 4: col 18 -> row 1
- U1 pad 5: col 15 -> row 2
- U1 pad 6: col 14 -> row 3
- U1 pad 7: col 13 -> row 4
- U1 pad 9: col 12 -> row 5
Routing:
- net col 17: track 603.5 -> 0.00 mm, vias 4 -> 0
- net col 18: track 587.4 -> 0.00 mm, vias 2 -> 0
- net encB: track 0.00 -> 372.1 mm, vias 0 -> 1
- net encA: track 0.00 -> 356.1 mm
- net row 4: track 529.2 -> 375.4 mm, vias 0 -> 1
- net col 10: track 426.9 -> 322.7 mm
- net row 3: track 482.7 -> 382.0 mm, vias 2 -> 1
- net row 5: track 534.8 -> 447.3 mm, vias 3 -> 1
- net col 12: track 468.4 -> 384.6 mm
- net col 11: track 450.4 -> 368.6 mm
- net row 2: track 447.1 -> 366.3 mm, vias 2 -> 1
- net col 9: track 344.0 -> 263.4 mm, vias 0 -> 2
- net col 15: track 504.1 -> 429.5 mm
- net col 13: track 476.4 -> 403.2 mm
- net col 14: track 491.6 -> 419.7 mm
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Other:
- board size 474.9 x 141 mm -> 395 x 121 mm
