File: PCB/hackboard.kicad_sch (KiCad schematic)
At the start: 204 parts, among them SW1 SW_Push_45deg, SW10 SW_Push_45deg, SW100 SW_Push_45deg, SW101 SW_Push_45deg, SW102 SW_Push_45deg, SW103 SW_Push_45deg, SW104 SW_Push_45deg, SW11 SW_Push_45deg, SW12 SW_Push_45deg, SW13 SW_Push_45deg, SW17 SW_Push_45deg, SW18 SW_Push_45deg, SW19 SW_Push_45deg, SW2 SW_Push_45deg, SW20 SW_Push_45deg, SW21 SW_Push_45deg, SW22 SW_Push_45deg, SW23 SW_Push_45deg, SW24 SW_Push_45deg, SW25 SW_Push_45deg, SW26 SW_Push_45deg, SW27 SW_Push_45deg, SW28 SW_Push_45deg, SW29 SW_Push_45deg, SW3 SW_Push_45deg, SW30 SW_Push_45deg, SW31 SW_Push_45deg, SW32 SW_Push_45deg, SW33 SW_Push_45deg, SW34 SW_Push_45deg, SW35 SW_Push_45deg, SW36 SW_Push_45deg, SW37 SW_Push_45deg, SW38 SW_Push_45deg, SW39 SW_Push_45deg, SW4 SW_Push_45deg, SW40 SW_Push_45deg, SW41 SW_Push_45deg, SW42 SW_Push_45deg, SW43 SW_Push_45deg, SW44 SW_Push_45deg, SW45 SW_Push_45deg, SW46 SW_Push_45deg, SW47 SW_Push_45deg, SW48 SW_Push_45deg, SW49 SW_Push_45deg, SW5 SW_Push_45deg, SW50 SW_Push_45deg, SW51 SW_Push_45deg, SW52 SW_Push_45deg, SW53 SW_Push_45deg, SW54 SW_Push_45deg, SW55 SW_Push_45deg, SW56 SW_Push_45deg, SW57 SW_Push_45deg, SW58 SW_Push_45deg, SW59 SW_Push_45deg, SW6 SW_Push_45deg, SW60 SW_Push_45deg, SW61 SW_Push_45deg, SW62 SW_Push_45deg, SW63 SW_Push_45deg, SW64 SW_Push_45deg, SW65 SW_Push_45deg, SW66 SW_Push_45deg, SW67 SW_Push_45deg, SW68 SW_Push_45deg, SW69 SW_Push_45deg, SW7 SW_Push_45deg, SW70 SW_Push_45deg, SW71 SW_Push_45deg, SW72 SW_Push_45deg, SW73 SW_Push_45deg, SW74 SW_Push_45deg, SW75 SW_Push_45deg, SW76 SW_Push_45deg, SW77 SW_Push_45deg, SW78 SW_Push_45deg, SW79 SW_Push_45deg, SW8 SW_Push_45deg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

Commit message: Add files via upload
Parts:
- removed D103, D33, D36, D37, D54, D57, D58, D74: 1N4148, Diode_SMD:D_SOD-123, symbol Diode:1N4148
- removed SW103: SW_Push_45deg, Button_Switch_Keyboard:SW_Cherry_MX_2.00u_PCB, symbol Switch:SW_Push_45deg
- removed SW33, SW36, SW37, SW54, SW57, SW74: SW_Push_45deg, Button_Switch_Keyboard:SW_Cherry_MX_1.00u_PCB, symbol Switch:SW_Push_45deg
- removed SW58: SW_Push_45deg, Button_Switch_Keyboard:SW_Cherry_MX_2.00u_Vertical_PCB, symbol Switch:SW_Push_45deg
- added D16, D90: 1N4148, Diode_SMD:D_SOD-123, symbol Diode:1N4148
- added SW1: RotaryEncoder_Switch, Rotary_Encoder:RotaryEncoder_Alps_EC11E-Switch_Vertical_H20mm, symbol Device:RotaryEncoder_Switch
- added SW90: SW_Push_45deg, Button_Switch_Keyboard:SW_Cherry_MX_1.25u_PCB, symbol Switch:SW_Push_45deg
- SW51: renamed from SW59; footprint Button_Switch_Keyboard:SW_Cherry_MX_1.75u_PCB -> Button_Switch_Keyboard:SW_Cherry_MX_2.00u_Vertical_PCB
- SW52: renamed from SW60; footprint Button_Switch_Keyboard:SW_Cherry_MX_1.00u_PCB -> Button_Switch_Keyboard:SW_Cherry_MX_1.75u_PCB
- SW63: renamed from SW71; footprint Button_Switch_Keyboard:SW_Cherry_MX_2.25u_PCB -> Button_Switch_Keyboard:SW_Cherry_MX_1.00u_PCB
- SW64: renamed from SW87; footprint Button_Switch_Keyboard:SW_Cherry_MX_1.00u_PCB -> Button_Switch_Keyboard:SW_Cherry_MX_2.25u_PCB
- SW67: renamed from SW75; footprint Button_Switch_Keyboard:SW_Cherry_MX_2.25u_PCB -> Button_Switch_Keyboard:SW_Cherry_MX_1.00u_PCB
- SW68: renamed from SW91; footprint Button_Switch_Keyboard:SW_Cherry_MX_2.00u_Vertical_PCB -> Button_Switch_Keyboard:SW_Cherry_MX_2.25u_PCB
- SW79: renamed from SW86; footprint Button_Switch_Keyboard:SW_Cherry_MX_2.75u_PCB -> Button_Switch_Keyboard:SW_Cherry_MX_1.75u_PCB
- SW81: renamed from SW88; footprint Button_Switch_Keyboard:SW_Cherry_MX_1.00u_PCB -> Button_Switch_Keyboard:SW_Cherry_MX_2.00u_PCB
- SW83: renamed from SW92; footprint Button_Switch_Keyboard:SW_Cherry_MX_1.25u_PCB -> Button_Switch_Keyboard:SW_Cherry_MX_1.00u_PCB
- SW84: renamed from SW104; footprint Button_Switch_Keyboard:SW_Cherry_MX_1.00u_PCB -> Button_Switch_Keyboard:SW_Cherry_MX_2.00u_Vertical_PCB
- SW86: renamed from SW94; footprint Button_Switch_Keyboard:SW_Cherry_MX_1.25u_PCB -> Button_Switch_Keyboard:SW_Cherry_MX_1.00u_PCB
- SW87: renamed from SW95; footprint Button_Switch_Keyboard:SW_Cherry_MX_1.25u_PCB -> Button_Switch_Keyboard:SW_Cherry_MX_1.00u_PCB
- SW88: renamed from SW97; footprint Button_Switch_Keyboard:SW_Cherry_MX_1.25u_PCB -> Button_Switch_Keyboard:SW_Cherry_MX_1.00u_PCB
- SW91: renamed from SW90; footprint Button_Switch_Keyboard:SW_Cherry_MX_1.00u_PCB -> Button_Switch_Keyboard:SW_Cherry_MX_1.25u_PCB
- SW92: renamed from SW98; footprint Button_Switch_Keyboard:SW_Cherry_MX_1.25u_PCB -> Button_Switch_Keyboard:SW_Cherry_MX_1.00u_PCB
- SW93: renamed from SW99; footprint Button_Switch_Keyboard:SW_Cherry_MX_1.25u_PCB -> Button_Switch_Keyboard:SW_Cherry_MX_1.00u_PCB
- renumbered D31 to D1, D8 to D10, D9 to D11, D10 to D12, D11 to D13, D12 to D14, D13 to D15, D52 to D17, D53 to D18, D17 to D19, D32 to D2, D18 to D20, D19 to D21, D20 to D22, D21 to D23, D22 to D24, D23 to D25, D24 to D26, D25 to D27, D26 to D28, D27 to D29, D1 to D3, D28 to D30, D29 to D31, D30 to D32, D34 to D33, D35 to D34, D38 to D35, D39 to D36, D40 to D37, D41 to D38, D42 to D39, D2 to D4, D43 to D40, D44 to D41, D45 to D42, D46 to D43, D47 to D44, D48 to D45, D49 to D46, D50 to D47, D51 to D48, D55 to D49, D3 to D5, D56 to D50, D59 to D51, D60 to D52, D61 to D53, D62 to D54, D63 to D55, D64 to D56, D65 to D57, D66 to D58, D67 to D59, D4 to D6, D68 to D60, D69 to D61, D70 to D62, D71 to D63, D87 to D64, D72 to D65, D73 to D66, D75 to D67, D91 to D68, D76 to D69, D5 to D7, D77 to D70, D78 to D71, D79 to D72, D80 to D73, D81 to D74, D82 to D75, D83 to D76, D84 to D77, D85 to D78, D86 to D79, D6 to D8, D101 to D80, D88 to D81, D89 to D82, D92 to D83, D104 to D84, D93 to D85, D94 to D86, D95 to D87, D97 to D88, D96 to D89, D7 to D9, D90 to D91, D98 to D92, D99 to D93, D100 to D94, D102 to D95, SW7 to SW10, SW8 to SW11, SW9 to SW12, SW10 to SW13, SW11 to SW14, SW12 to SW15, SW13 to SW16, SW52 to SW17, SW53 to SW18, SW17 to SW19, SW31 to SW2, SW18 to SW20, SW19 to SW21, SW20 to SW22, SW21 to SW23, SW22 to SW24, SW23 to SW25, SW24 to SW26, SW25 to SW27, SW26 to SW28, SW27 to SW29, SW32 to SW3, SW28 to SW30, SW29 to SW31, SW30 to SW32, SW34 to SW33, SW35 to SW34, SW38 to SW35, SW39 to SW36, SW40 to SW37, SW41 to SW38, SW42 to SW39, SW1 to SW4, SW43 to SW40, SW44 to SW41, SW45 to SW42, SW46 to SW43, SW47 to SW44, SW48 to SW45, SW49 to SW46, SW50 to SW47, SW51 to SW48, SW55 to SW49, SW2 to SW5, SW56 to SW50, SW61 to SW53, SW62 to SW54, SW63 to SW55, SW64 to SW56, SW65 to SW57, SW66 to SW58, SW67 to SW59, SW3 to SW6, SW68 to SW60, SW69 to SW61, SW70 to SW62, SW72 to SW65, SW73 to SW66, SW76 to SW69, SW4 to SW7, SW77 to SW70, SW78 to SW71, SW79 to SW72, SW80 to SW73, SW81 to SW74, SW82 to SW75, SW83 to SW76, SW84 to SW77, SW85 to SW78, SW5 to SW8, SW101 to SW80, SW89 to SW82, SW93 to SW85, SW96 to SW89, SW6 to SW9, SW100 to SW94, SW102 to SW95
Connections:
- net GND: now also U1.28 (GND), SW1.C; no longer U1.38 (GND)
- net clock: now also U1.32 (GPIO27_ADC1); no longer U1.2 (GPIO1)
- net col 1: now also SW17.1, SW2.1, SW33.1, SW49.1, SW65.1, SW81.1, U1.2 (GPIO1); no longer SW19.1, SW35.1, SW4.1, SW51.1, SW67.1, SW83.1, U1.34 (GPIO28_ADC2)
- net col 10: now also SW11.1, SW26.1, SW42.1, SW58.1, SW74.1, SW89.1; no longer SW13.1, SW28.1, SW44.1, SW60.1, SW76.1, SW88.1
- net col 11: now also SW12.1, SW27.1, SW43.1, SW59.1, SW75.1, U1.12 (GPIO9), SW90.1; no longer SW14.1, SW29.1, SW45.1, SW61.1, SW77.1, SW92.1, U1.10 (GPIO7)
- net col 12: now also SW13.1, SW28.1, SW44.1, SW60.1, SW76.1, SW91.1, U1.26 (GPIO20); no longer SW15.1, SW30.1, SW46.1, SW62.1, SW78.1, SW93.1, U1.9 (GPIO6)
- net col 13: now also SW14.1, SW29.1, SW45.1, SW61.1, SW77.1, SW92.1, U1.25 (GPIO19); no longer SW16.1, SW31.1, SW47.1, SW63.1, SW79.1, SW94.1, U1.7 (GPIO5)
- net col 14: now also SW15.1, SW30.1, SW46.1, SW62.1, SW78.1, SW93.1, U1.24 (GPIO18); no longer SW32.1, SW48.1, SW64.1, SW80.1, SW95.1, U1.6 (GPIO4)
- net col 15: now also SW16.1, SW31.1, SW47.1, SW63.1, SW79.1, SW94.1, U1.22 (GPIO17); no longer SW17.1, SW2.1, SW33.1, SW49.1, SW65.1, SW81.1, U1.5 (GPIO3)
- net col 16: now also SW32.1, SW48.1, SW64.1, SW80.1, SW95.1, U1.21 (GPIO16), SW1.S2; no longer SW18.1, SW3.1, SW34.1, SW50.1, SW66.1, SW82.1, U1.14 (GPIO10)
- net col 2: now also SW18.1, SW3.1, SW34.1, SW50.1, SW66.1, SW82.1, U1.10 (GPIO7); no longer SW20.1, SW36.1, SW5.1, SW52.1, U1.22 (GPIO17)
- net col 3: now also SW19.1, SW35.1, SW4.1, SW51.1, SW67.1, SW83.1, U1.27 (GPIO21); no longer SW21.1, SW37.1, SW53.1, SW6.1, SW69.1, SW85.1, U1.31 (GPIO26_ADC0)
- net col 4: now also SW20.1, SW36.1, SW5.1, SW52.1, SW68.1, SW84.1, U1.14 (GPIO10); no longer SW22.1, SW38.1, SW54.1, SW7.1, SW70.1, SW86.1, U1.29 (GPIO22)
- net col 5: now also SW21.1, SW37.1, SW53.1, SW6.1, SW69.1, SW85.1, U1.15 (GPIO11); no longer SW23.1, SW39.1, SW55.1, SW71.1, SW8.1, SW87.1, U1.25 (GPIO19)
- net col 6: now also SW22.1, SW38.1, SW54.1, SW7.1, SW70.1, SW86.1, U1.16 (GPIO12); no longer SW24.1, SW40.1, SW56.1, SW72.1, SW9.1, U1.26 (GPIO20)
- net col 7: now also SW23.1, SW39.1, SW55.1, SW71.1, SW8.1, SW87.1, U1.17 (GPIO13); no longer SW10.1, SW25.1, SW41.1, SW57.1, SW73.1, U1.27 (GPIO21)
- net col 8: now also SW24.1, SW40.1, SW56.1, SW72.1, SW88.1, SW9.1, U1.19 (GPIO14); no longer SW11.1, SW26.1, SW42.1, SW58.1, SW74.1, SW89.1, U1.15 (GPIO11)
- net col 9: now also SW10.1, SW25.1, SW41.1, SW57.1, SW73.1, U1.20 (GPIO15); no longer SW12.1, SW27.1, SW43.1, SW59.1, SW75.1, U1.12 (GPIO9)
- net data: now also U1.31 (GPIO26_ADC0); no longer U1.1 (GPIO0)
- net row 1: now also U1.4 (GPIO2), D16.1 (K); no longer U1.32 (GPIO27_ADC1)
- net row 2: now also U1.5 (GPIO3); no longer U1.24 (GPIO18)
- net row 3: now also U1.6 (GPIO4); no longer U1.16 (GPIO12)
- net row 4: now also U1.7 (GPIO5); no longer D68.1 (K), U1.17 (GPIO13)
- net row 5: now also D68.1 (K), U1.9 (GPIO6); no longer D84.1 (K), U1.19 (GPIO14)
- net row 6: now also D84.1 (K), U1.1 (GPIO0), D90.1 (K); no longer U1.20 (GPIO15)
- net at D2.2 (A): now also SW2.2; no longer SW3.2
- net at D9.2 (A): now also SW9.2; no longer SW10.2
- net at SW16.2: now also D16.2 (A); no longer D15.2 (A)
- net at D13.2 (A): now also SW13.2; no longer SW14.2
- net at D7.2 (A): now also SW7.2; no longer SW8.2
- net at D10.2 (A): now also SW10.2; no longer SW11.2
- net at D11.2 (A): now also SW11.2; no longer SW12.2
- net at SW4.2: now also D4.2 (A); no longer D3.2 (A)
- net at D5.2 (A): now also SW5.2; no longer SW6.2
- net at D8.2 (A): now also SW8.2; no longer SW9.2
- net at SW15.2: now also D15.2 (A); no longer D14.2 (A)
- net at D12.2 (A): now also SW12.2; no longer SW13.2
- net at D6.2 (A): now also SW6.2; no longer SW7.2
- net at D1.2 (A): now also SW1.S1; no longer SW2.2
- removed net col 17: SW91.1, U1.21 (GPIO16)
- removed net col 18: SW68.1, SW84.1, U1.4 (GPIO2)
- new net: D3.2 (A), SW3.2
- new net: D90.2 (A), SW90.2
- new net: D14.2 (A), SW14.2
- new net encA: SW1.B, U1.29 (GPIO22)
- new net encB: SW1.A, U1.34 (GPIO28_ADC2)
Other:
- moved on the sheet: D1, D10, D11, D12, D13, D14, D15, D17, D18, D19, D2, D20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
